Commit message: Setup centered robot base

File: nav_sim_c/models/differential_robot.urdf (robot description, URDF)
Before this commit: robot differential_robot, 2 links, 1 joints
Links:
- link base_link: geometry visual box size=${base_inner_width} ${base_length} ${base_height}

Commit message: Fixed base link and footprint offset

File: nav_sim_c/models/differential_robot.urdf (robot description, URDF)
Before this commit: robot differential_robot, 2 links, 1 joints
Joints:
- joint base_joint: origin xyz=0.0 0.0 ${-(wheel_radius+wheel_zoff)} rpy=0 0 0 -> xyz=0.0 0.0 ${-(base_height / 2 + base_ground_height_zoffset)} rpy=0 0 0

Commit message: Added interial to base and fixed tabbing

File: nav_sim_c/models/differential_robot.urdf (robot description, URDF)
Before this commit: robot differential_robot, 2 links, 1 joints
Links:
- link base_link: geometry collision box size=${base_inner_width} ${base_length} ${base_height}; visual box size=${base_inner_width} ${base_length} ${base_height}

Commit message: Added simulated ros gazebo imu

File: nav_sim_c/models/differential_robot.urdf (robot description, URDF)
Before this commit: robot differential_robot, 2 links, 1 joints
Links:
- added link imu_link; collision box size=0.1 0.1 0.1; visual box size=0.1 0.1 0.1
Joints:
- added joint imu_joint: type fixed, parent base_link, child imu_link, origin xyz=0 0 0.01
